File: kicad/218-pdb.kicad_pcb (KiCad board)
At the start: 2 copper layers, 80 x 55.4 mm, 73 parts, among them J1 Conn_01x03, J10 Conn_01x03, J11 Conn_01x03, J12 Conn_01x03, J13 Conn_01x03, J14 Conn_01x03, J15 Conn_01x03, J16 Conn_01x03, J17 Conn_01x03, J18 Conn_01x03, J19 Conn_01x03, J2 Conn_01x03, J20 Conn_01x03, J21 Conn_01x03, J22 Conn_01x03, J23 Conn_01x03, J24 Conn_01x03, J25 Conn_01x04_Pin, J26 Conn_01x04_Pin, J27 Conn_01x04_Pin, J28 Conn_01x04_Pin, J29 14 V molex, J3 Conn_01x03, J30 14 V molex, J31 14 V molex, J32 14 V molex, J33 external 5V, J34 battery, J35 battery, J4 Conn_01x03, J5 Conn_01x03, J6 Conn_01x03, J7 Conn_01x03, J8 Conn_01x03, J9 Conn_01x03, SW1 5V switch, U1 DC-DC buck, U2 DC-DC buck, U3 LD1117V33, U4 LD1117V33

Commit message: change diode
Parts:
- D6: value schottky diode, >=2 Amp -> diode, >=2 Amp; footprint Diode_THT:D_DO-41_SOD81_P2.54mm_Vertical_AnodeUp -> Diode_THT:D_DO-15_P2.54mm_Vertical_AnodeUp
Routing:
- net 14-1: track 19.5 -> 24.8 mm
- net GND: track 102.2 -> 107.3 mm
Other:
- board text added: "Batteries"
- board text removed: "Battery"

Commit message: update silkscreen
Other:
- board text added: "1"
- board text added: "10"
- board text added: "11"
- board text added: "12"
- board text added: "13"
- board text added: "14"
- board text added: "15"
- board text added: "16"
- board text added: "2"
- board text added: "3"
- board text added: "4"
- board text added: "5"
- board text added: "6"
- board text added: "7"
- board text added: "8"
- board text added: "9"

Commit message: update silkscreen
Parts:
- main1: value MotorSW -> MainSW
Other:
- board text added: "17 18 19 20 21 22 23 24"
- board text added: "main"
- board text removed: "motor"
Changed lines of the file:
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@@
 		(tags "Through hole pin header THT 1x03 2.54mm single row")
 		(property "Reference" "NT2"
-			(at -0.254 -2.032 90)
+			(at 0.0254 -2.2098 90)
 			(layer "F.SilkS")
 			(effects
@@
 			)
 		)
-		(property "Value" "MotorSW"
+		(property "Value" "MainSW"
 			(at 8.382 0.762 0)
 			(layer "F.SilkS")
@@
 	)
 	(gr_line
+		(start 140.2588 81.8896)
+		(end 140.859996 82.815378)
+		(stroke
+			(width 0.1)
+			(type default)
+		)
+		(layer "F.SilkS")
+	)
+	(gr_line
 		(start 98.552 86.9188)
 		(end 98.9584 88.5952)
@@
 		)
 	)
-	(gr_text "motor"
-		(at 139.936904 89.390093 0)
+	(gr_text "main"
+		(at 139.192 89.408 0)
 		(layer "F.SilkS")
 		(effects
@@
 		)
 	)
+	(gr_text "17        18        19        20        21        22        23        24 "
+		(at 81.3816 67.1576 0)
+		(layer "F.SilkS")
+		(effects
+			(font
+				(size 1 0.94)
+				(thickness 0.1125)
+			)
+			(justify left bottom)
+		)
+	)
 	(gr_text "5V"
 		(at 146.12902 89.446861 0)
@@
 	)
 	(gr_text "servo"
-		(at 138.938 90.932 90)
+		(at 138.684 91.6432 90)
 		(layer "F.SilkS")
 		(effects
@@
 	)
 	(zone
-		(net 27)
-		(net_name "Net-(NT1-A)")
+		(net 18)
+		(net_name "5-2")
 		(layer "F.Cu")
 		(name "$teardrop_padvia$")
 		(hatch none 0.1)
-		(priority 30008)
+		(priority 30001)
 		(attr
 			(teardrop
@@
 		(polygon
 			(pts
-				(xy 138.838812 58.896562) (xy 138.485258 59.250116) (xy 138.946613 60.051437) (xy 139.363055 59.774359)
-				(xy 139.640133 59.357917)
+				(xy 109.343 58.969136) (xy 108.843 58.969136) (xy 108.602607 59.861984) (xy 109.093 59.960529) (xy 109.583393 59.861984)
 			)
 		)
@@
 	)
 	(zone
-		(net 18)
-		(net_name "5-2")
+		(net 27)
+		(net_name "Net-(NT1-A)")
 		(layer "F.Cu")
 		(name "$teardrop_padvia$")
 		(hatch none 0.1)
-		(priority 30003)
+		(priority 30008)
 		(attr
 			(teardrop
@@
 		(polygon
 			(pts
-				(xy 108.836607 70.545973) (xy 109.336607 70.545973) (xy 109.577 69.653125) (xy 109.086607 69.55458)
-				(xy 108.596214 69.653125)
+				(xy 138.838812 58.896562) (xy 138.485258 59.250116) (xy 138.946613 60.051437) (xy 139.363055 59.774359)
+				(xy 139.640133 59.357917)
 			)
 		)
 	)
 	(zone
-		(net 27)
-		(net_name "Net-(NT1-A)")
+		(net 18)
+		(net_name "5-2")
 		(layer "F.Cu")
 		(name "$teardrop_padvia$")
 		(hatch none 0.1)
-		(priority 30007)
+		(priority 30002)
 		(attr
 			(teardrop
@@
 		(polygon
 			(pts
-				(xy 139.320955 72.044393) (xy 139.820955 72.044393) (xy 140.061348 71.151545) (xy 139.570955 71.053)
-				(xy 139.080562 71.151545)
+				(xy 108.836607 70.545973) (xy 109.336607 70.545973) (xy 109.577 69.653125) (xy 109.086607 69.55458)
+				(xy 108.596214 69.653125)
 			)
 		)
@@
 		(name "$teardrop_padvia$")
 		(hatch none 0.1)
-		(priority 30001)
+		(priority 30005)
 		(attr
 			(teardrop
@@
 		(polygon
 			(pts
-				(xy 109.343 58.969136) (xy 108.843 58.969136) (xy 108.602607 59.861984) (xy 109.093 59.960529) (xy 109.583393 59.861984)
+				(xy 108.836607 62.849922) (xy 109.336607 62.849922) (xy 109.583393 61.957074) (xy 109.093 61.858529)
+				(xy 108.602607 61.957074)
 			)
 		)
@@
 		(name "$teardrop_padvia$")
 		(hatch none 0.1)
-		(priority 30002)
+		(priority 30004)
 		(attr
 			(teardrop
@@
 		(polygon
 			(pts
-				(xy 109.336607 71.745187) (xy 108.836607 71.745187) (xy 108.600442 72.638035) (xy 109.090835 72.73658)
-				(xy 109.581228 72.638035)
+				(xy 109.336607 66.665187) (xy 108.836607 66.665187) (xy 108.596214 67.558035) (xy 109.086607 67.65658)
+				(xy 109.577 67.558035)
 			)
 		)
 	)
 	(zone
-		(net 18)
-		(net_name "5-2")
+		(net 27)
+		(net_name "Net-(NT1-A)")
 		(layer "F.Cu")
 		(name "$teardrop_padvia$")
 		(hatch none 0.1)
-		(priority 30004)
+		(priority 30006)
 		(attr
 			(teardrop
@@
 		(polygon
 			(pts
-				(xy 109.336607 66.665187) (xy 108.836607 66.665187) (xy 108.596214 67.558035) (xy 109.086607 67.65658)
-				(xy 109.577 67.558035)
+				(xy 139.069 63.093393) (xy 139.569 63.093393) (xy 139.809393 62.200545) (xy 139.319 62.102) (xy 138.828607 62.200545)
 			)
 		)
@@
 	)
 	(zone
-		(net 18)
-		(net_name "5-2")
+		(net 27)
+		(net_name "Net-(NT1-A)")
 		(layer "F.Cu")
 		(name "$teardrop_padvia$")
 		(hatch none 0.1)
-		(priority 30005)
+		(priority 30007)
 		(attr
 			(teardrop
@@
 		(polygon
 			(pts
-				(xy 108.836607 62.849922) (xy 109.336607 62.849922) (xy 109.583393 61.957074) (xy 109.093 61.858529)
-				(xy 108.602607 61.957074)
+				(xy 139.320955 72.044393) (xy 139.820955 72.044393) (xy 140.061348 71.151545) (xy 139.570955 71.053)
+				(xy 139.080562 71.151545)
 			)
 		)
@@
 	)
 	(zone
+		(net 18)
+		(net_name "5-2")
+		(layer "F.Cu")
+		(name "$teardrop_padvia$")
+		(hatch none 0.1)
+		(priority 30003)
+		(attr
+			(teardrop
+				(type padvia)
+			)
+		)
+		(connect_pads yes
+			(clearance 0)
+		)
+		(min_thickness 0.0254)
+		(filled_areas_thickness no)
+		(fill yes
+			(thermal_gap 0.5)
+			(thermal_bridge_width 0.5)
+			(island_removal_mode 1)
+			(island_area_min 10)
+		)
+		(polygon
+			(pts
+				(xy 109.336607 71.745187) (xy 108.836607 71.745187) (xy 108.600442 72.638035) (xy 109.090835 72.73658)
+				(xy 109.581228 72.638035)
+			)
+		)
+	)
+	(zone
 		(net 14)
 		(net_name "+BATT")
@@
 	)
 	(zone
-		(net 27)
-		(net_name "Net-(NT1-A)")
-		(layer "F.Cu")
+		(net 18)
+		(net_name "5-2")
+		(layer "B.Cu")
 		(name "$teardrop_padvia$")
 		(hatch none 0.1)
-		(priority 30006)
+		(priority 30003)
 		(attr
 			(teardrop
@@
 		(polygon
 			(pts
-				(xy 139.069 63.093393) (xy 139.569 63.093393) (xy 139.809393 62.200545) (xy 139.319 62.102) (xy 138.828607 62.200545)
+				(xy 108.836607 68.645973) (xy 109.336607 68.645973) (xy 109.577 67.753125) (xy 109.086607 67.65458)
+				(xy 108.596214 67.753125)
 			)
 		)
@@
 		(polygon
 			(pts
-				(xy 139.820955 70.063607) (xy 139.320955 70.063607) (xy 139.080562 70.956455) (xy 139.570955 71.055)
-				(xy 140.061348 70.956455)
-			)
-		)
-	)
-	(zone
-		(net 27)
-		(net_name "Net-(NT1-A)")
-		(layer "B.Cu")
-		(name "$teardrop_padvia$")
-		(hatch none 0.1)
-		(priority 30009)
-		(attr
-			(teardrop
-				(type padvia)
-			)
-		)
-		(connect_pads yes
-			(clearance 0)
-		)
-		(min_thickness 0.0254)
-		(filled_areas_thickness no)
-		(fill yes
-			(thermal_gap 0.5)
-			(thermal_bridge_width 0.5)
-			(island_removal_mode 1)
-			(island_area_min 10)
-		)
-		(polygon
-			(pts
-				(xy 139.696 61.124808) (xy 139.196 61.124808) (xy 138.903265 61.825215) (xy 139.319 62.104) (xy 139.809393 62.005455)
+				(xy 139.320955 69.189393) (xy 139.820955 69.189393) (xy 140.063393 68.296545) (xy 139.573 68.198)
+				(xy 139.082607 68.296545)
 			)
 		)
@@
 		(polygon
 			(pts
-				(xy 109.340835 73.645187) (xy 108.840835 73.645187) (xy 108.600442 74.538035) (xy 109.090835 74.63658)
-				(xy 109.581228 74.538035)
+				(xy 108.840835 73.725973) (xy 109.340835 73.725973) (xy 109.581228 72.833125) (xy 109.090835 72.73458)
+				(xy 108.600442 72.833125)
 			)
 		)
 	)
 	(zone
-		(net 27)
-		(net_name "Net-(NT1-A)")
+		(net 18)
+		(net_name "5-2")
 		(layer "B.Cu")
 		(name "$teardrop_padvia$")
 		(hatch none 0.1)
-		(priority 30008)
+		(priority 30002)
 		(attr
 			(teardrop
@@
 		(polygon
 			(pts
-				(xy 139.196 60.764045) (xy 139.696 60.764045) (xy 139.852741 59.871197) (xy 139.362348 59.772652)
-				(xy 138.871955 59.871197)
+				(xy 109.336607 68.565187) (xy 108.836607 68.565187) (xy 108.596214 69.458035) (xy 109.086607 69.55658)
+				(xy 109.577 69.458035)
 			)
 		)
@@
 		(name "$teardrop_padvia$")
 		(hatch none 0.1)
-		(priority 30005)
+		(priority 30004)
 		(attr
 			(teardrop
@@
 		(polygon
 			(pts
-				(xy 108.840835 73.725973) (xy 109.340835 73.725973) (xy 109.581228 72.833125) (xy 109.090835 72.73458)
-				(xy 108.600442 72.833125)
+				(xy 109.340835 73.645187) (xy 108.840835 73.645187) (xy 108.600442 74.538035) (xy 109.090835 74.63658)
+				(xy 109.581228 74.538035)
 			)
 		)
 	)
 	(zone
-		(net 18)
-		(net_name "5-2")
+		(net 27)
+		(net_name "Net-(NT1-A)")
 		(layer "B.Cu")
 		(name "$teardrop_padvia$")
 		(hatch none 0.1)
-		(priority 30004)
+		(priority 30009)
 		(attr
 			(teardrop
@@
 		(polygon
 			(pts
-				(xy 109.343 60.869136) (xy 108.843 60.869136) (xy 108.602607 61.761984) (xy 109.093 61.860529) (xy 109.583393 61.761984)
+				(xy 139.696 61.124808) (xy 139.196 61.124808) (xy 138.903265 61.825215) (xy 139.319 62.104) (xy 139.809393 62.005455)
 			)
 		)
 	)
 	(zone
-		(net 18)
-		(net_name "5-2")
+		(net 27)
+		(net_name "Net-(NT1-A)")
 		(layer "B.Cu")
 		(name "$teardrop_padvia$")
 		(hatch none 0.1)
-		(priority 30002)
+		(priority 30008)
 		(attr
 			(teardrop
@@
 		(polygon
 			(pts
-				(xy 108.836607 68.645973) (xy 109.336607 68.645973) (xy 109.577 67.753125) (xy 109.086607 67.65458)
-				(xy 108.596214 67.753125)
+				(xy 139.196 60.764045) (xy 139.696 60.764045) (xy 139.852741 59.871197) (xy 139.362348 59.772652)
+				(xy 138.871955 59.871197)
 			)
 		)
 	)
 	(zone
-		(net 27)
-		(net_name "Net-(NT1-A)")
+		(net 18)
+		(net_name "5-2")
 		(layer "B.Cu")
 		(name "$teardrop_padvia$")
 		(hatch none 0.1)
-		(priority 30007)
+		(priority 30005)
 		(attr
 			(teardrop
@@
 		(polygon
 			(pts
-				(xy 139.320955 69.189393) (xy 139.820955 69.189393) (xy 140.063393 68.296545) (xy 139.573 68.198)
-				(xy 139.082607 68.296545)
+				(xy 109.343 60.869136) (xy 108.843 60.869136) (xy 108.602607 61.761984) (xy 109.093 61.860529) (xy 109.583393 61.761984)
 			)
 		)
 	)
 	(zone
-		(net 18)
-		(net_name "5-2")
+		(net 27)
+		(net_name "Net-(NT1-A)")
 		(layer "B.Cu")
 		(name "$teardrop_padvia$")
 		(hatch none 0.1)
-		(priority 30003)
+		(priority 30007)
 		(attr
 			(teardrop
@@
 		(polygon
 			(pts
-				(xy 109.336607 68.565187) (xy 108.836607 68.565187) (xy 108.596214 69.458035) (xy 109.086607 69.55658)
-				(xy 109.577 69.458035)
+				(xy 139.820955 70.063607) (xy 139.320955 70.063607) (xy 139.080562 70.956455) (xy 139.570955 71.055)
+				(xy 140.061348 70.956455)
 			)
 		)

Commit message: restart
Parts:
- removed C5: 10 uF, Capacitor_THT:C_Disc_D3.8mm_W2.6mm_P2.50mm
- removed FID5, FID6, FID7, FID8: one header pin, 218-pdb:PinHeader_1x01_P2.54mm_Vertical
- removed J34, J35: battery, 218-pdb:CUI_TB007-508-02BE
- added C3: 0.1 uF, Capacitor_THT:C_Disc_D3.0mm_W2.0mm_P2.50mm, F.Cu at (278.9, 121.1)
- added U5: LD1117V50, 218-pdb:TO255P1020X450X1968-3, F.Cu at (244.1, 122.0)
- C2: value 0.1 uF -> 10 uF; footprint Capacitor_THT:C_Disc_D3.0mm_W2.0mm_P2.50mm -> Capacitor_THT:C_Disc_D3.8mm_W2.6mm_P2.50mm
- FID1, FID2: value jumper -> one 90 degree header pin; footprint 218-pdb:jumper -> 218-pdb:PinHeader_1x01_P2.54mm_H
- FID10, FID9: value one header pin -> jumper; footprint 218-pdb:PinHeader_1x01_P2.54mm_Vertical -> 218-pdb:jumper
- FID3, FID4: value one header pin -> one 90 degree header pin; footprint 218-pdb:PinHeader_1x01_P2.54mm_Vertical -> 218-pdb:PinHeader_1x01_P2.54mm_H; moved to F.Cu
- J1, J10, J11, J12, J13, J14, J15, J16, J2, J3, J4, J5, J6, J7, J8, J9: footprint 218-pdb:Molex_KK-254_AE-6410-03A_1x03_P2.54mm_Vertical -> 218-pdb:JST_XH_B3B-XH-A_1x03_P2.50mm_Vertical
- J27: value Conn_01x04_Pin -> external 5V; footprint Connector_PinHeader_2.54mm:PinHeader_1x04_P2.54mm_Vertical -> 218-pdb:Molex_KK-254_AE-6410-02A_1x02_P2.54mm_Vertical
- J28: value Conn_01x04_Pin -> battery; footprint Connector_PinHeader_2.54mm:PinHeader_1x04_P2.54mm_Vertical -> 218-pdb:CUI_TB007-508-02BE
- J29, J30, J31, J32: value 14 V molex -> battery; footprint 218-pdb:Molex_KK-396_A-41791-0002_1x02_P3.96mm_Vertical -> 218-pdb:CUI_TB007-508-02BE
- J33: value external 5V -> battery; footprint 218-pdb:Molex_KK-254_AE-6410-02A_1x02_P2.54mm_Vertical -> 218-pdb:CUI_TB007-508-02BE
- R2: value 680 -> 1k
- R3: value 3.3k -> 680
- R5: value 1k -> 3.3k
- U1: value DC-DC buck -> LD1117V33; footprint 218-pdb:HW-411 -> 218-pdb:TO255P1020X450X1968-3; moved to F.Cu
- U2: moved to F.Cu
- U4: value LD1117V33 -> DC-DC buck; footprint 218-pdb:TO255P1020X450X1968-3 -> 218-pdb:HW-411
- moved FID9 186.3 mm to (273.4, 119.7), turned to 0 degrees
- moved main1 184.8 mm to (264.4, 100.3), turned to 0 degrees
- moved J9 183.7 mm to (265.1, 53.6), turned to 0 degrees
- moved J10 175.4 mm to (265.1, 61.4), turned to 0 degrees
- moved FID10 173.3 mm to (276.8, 126.7), turned to 180 degrees
- moved J25 171.1 mm to (252.3, 118.1), turned to 0 degrees
- moved J11 167.4 mm to (265.1, 69.2), turned to 0 degrees
- moved J13 165.3 mm to (277.0, 53.6), turned to 0 degrees
- moved J12 159.7 mm to (265.1, 77.0), turned to 0 degrees
- moved J1 159.0 mm to (241.2, 53.6), turned to 0 degrees
- moved J14 156.9 mm to (277.0, 61.4), turned to 0 degrees
- moved J26 153.2 mm to (256.9, 118.1), turned to 0 degrees
- moved J2 151.0 mm to (241.2, 61.4), turned to 0 degrees
- moved J27 151.0 mm to (267.1, 119.8), turned to 0 degrees
- moved TP1 149.5 mm to (251.7, 129.8)
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Connections:
- C2 pad 1: 5-1 -> 3.3-1
- C4 pad 1: 3.3-1 -> 3.3-2
- D2 pad 2: 3.3-2 -> 5-2
- D3 pad 2: 14-3 -> 3.3-2
- D5 pad 2: 5-2 -> 14-3
- J1 pad 1: GND -> 3.3-1
- J1 pad 2: 3.3-1 -> GND
- J1 pad 3: Net-(J1-Pin_3) -> 5-1
- J2 pad 1: GND -> 3.3-1
- J2 pad 2: 3.3-1 -> GND
- J2 pad 3: Net-(J2-Pin_3) -> 5-1
- J25 pad 1: Net-(J1-Pin_3) -> Net-(J17-Pin_3)
- J25 pad 2: Net-(J2-Pin_3) -> Net-(J18-Pin_3)
- J25 pad 3: Net-(J25-Pin_3) -> Net-(J19-Pin_3)
- J25 pad 4: Net-(J25-Pin_4) -> Net-(J20-Pin_3)
- J26 pad 1: Net-(J26-Pin_1) -> Net-(J21-Pin_3)
- J26 pad 2: Net-(J26-Pin_2) -> Net-(J22-Pin_3)
- J26 pad 3: Net-(J26-Pin_3) -> Net-(J23-Pin_3)
- J26 pad 4: Net-(J26-Pin_4) -> Net-(J24-Pin_3)
- J27 pad 1: Net-(J21-Pin_3) -> GND
- J27 pad 2: Net-(J22-Pin_3) -> Net-(J27-Pin_2)
- J28 pad 1: Net-(J17-Pin_3) -> GND
- J28 pad 2: Net-(J18-Pin_3) -> 14-3
- J3 pad 1: GND -> 3.3-1
- J3 pad 2: 3.3-1 -> GND
- J3 pad 3: Net-(J25-Pin_3) -> 5-1
- J32 pad 1: GND -> +BATT
- J32 pad 2: 14-3 -> Net-(J32-Pin_2)
- J33 pad 1: GND -> Net-(J32-Pin_2)
- J33 pad 2: Net-(J33-Pin_2) -> GND
- J4 pad 1: GND -> 3.3-1
- J4 pad 2: 3.3-1 -> GND
- J4 pad 3: Net-(J25-Pin_4) -> 5-1
- J5 pad 1: GND -> 3.3-1
- J5 pad 2: 3.3-1 -> GND
- J5 pad 3: Net-(J26-Pin_1) -> 5-1
- J6 pad 1: GND -> 3.3-1
- J6 pad 2: 3.3-1 -> GND
- J6 pad 3: Net-(J26-Pin_2) -> 5-1
- J7 pad 1: GND -> 3.3-1
- J7 pad 2: 3.3-1 -> GND
- J7 pad 3: Net-(J26-Pin_3) -> 5-1
- J8 pad 1: GND -> 3.3-1
- J8 pad 2: 3.3-1 -> GND
- J8 pad 3: Net-(J26-Pin_4) -> 5-1
- NT1 pad 2: 5-1 -> Net-(NT1-B)
- NT1 pad 3: Net-(J33-Pin_2) -> Net-(J27-Pin_2)
- U1 pad 1: 14-1 -> GND
- U1 pad 2: GND -> 3.3-1
- U1 pad 3: GND -> 5-1
- U3 pad 2: 3.3-1 -> 3.3-2
- U4 pad 1: GND -> 14-1
- U4 pad 2: 3.3-2 -> GND
- U4 pad 3: 5-1 -> GND
Routing:
- net 5-2: track 114.9 -> 0.00 mm, vias 6 -> 0
- net 5-1: track 109.4 -> 0.00 mm
- net GND: track 107.3 -> 0.00 mm
- net +BATT: track 86.6 -> 0.00 mm
- net 14-3: track 83.6 -> 0.00 mm
- net 3.3-2: track 75.4 -> 0.00 mm
- net 3.3-1: track 69.9 -> 0.00 mm
- net 14-2: track 39.3 -> 0.00 mm
- net Net-(NT1-A): track 33.1 -> 0.00 mm, vias 4 -> 0
- net 14-1: track 24.8 -> 0.00 mm
- net Net-(D3-K): track 6.21 -> 0.00 mm
- net Net-(D4-K): track 4.49 -> 0.00 mm
- net Net-(D5-K): track 4.47 -> 0.00 mm
- net Net-(D2-K): track 3.44 -> 0.00 mm
- net Net-(D1-K): track 3.42 -> 0.00 mm
- removed copper zone on F.Cu, net +BATT
- removed copper zone on F.Cu, net 14-3
- removed copper zone on B.Cu, net GND
- removed copper zone on F.Cu, net Net-(J34-Pin_2)
Other:
- board outline removed
- board text removed: "+"
- board text removed: "+ -"
- board text removed: "+ - + -"
- board text removed: "-"
- board text removed: "1"
- board text removed: "10"
- board text removed: "11"
- board text removed: "12"
- board text removed: "13"
- board text removed: "14"
- board text removed: "15"
- board text removed: "16"
- board text removed: "17 18 19 20 21 22 23 24"
- board text removed: "2"
- board text removed: "3"
- board text removed: "4"
- board text removed: "5"
- board text removed: "5 G 3"
- board text removed: "5V"
- board text removed: "6"
- board text removed: "7"
- board text removed: "8"
- board text removed: "9"
- board text removed: "Batteries"
- board text removed: "G 5 S"
- board text removed: "PIC DC-DC"
- board text removed: "S 3 G"
- board text removed: "SPDL PDB"
- board text removed: "Servo DC-DC"
- board text removed: "ext."
- board text removed: "main"
- board text removed: "on"
- board text removed: "servo"
- board text removed: "switch"
- board text removed: "v2.0 2026"

Commit message: start design E
Parts:
- added C5: 10 uF, Capacitor_THT:C_Disc_D3.8mm_W2.6mm_P2.50mm, F.Cu at (77.5, 167.7)
- added C6: 0.1 uF, Capacitor_THT:C_Disc_D3.0mm_W2.0mm_P2.50mm, F.Cu at (77.5, 163.8)
- moved FID9 217.6 mm to (58.5, 153.6)
- moved NT1 217.6 mm to (58.4, 151.1)
- moved D4 194.1 mm to (29.0, 156.2)
- moved R4 194.1 mm to (35.6, 153.7)
- moved J27 183.4 mm to (87.6, 157.5)
- moved J26 182.4 mm to (80.0, 73.7), turned to 180 degrees
- moved J25 172.9 mm to (80.0, 104.1), turned to 180 degrees
- moved J9 169.7 mm to (96.5, 73.6), turned to 90 degrees
- moved U5 167.5 mm to (79.3, 151.5), turned to 90 degrees
- moved J10 161.4 mm to (104.1, 73.6), turned to 90 degrees
- moved J11 153.4 mm to (111.8, 73.6), turned to 90 degrees
- moved J13 151.3 mm to (127.0, 73.6), turned to 90 degrees
- moved J12 145.7 mm to (119.4, 73.6), turned to 90 degrees
- moved J1 144.8 mm to (96.5, 60.9), turned to 90 degrees
- moved H2 144.5 mm to (80.0, 54.6)
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Connections:
- J1 pad 1: 3.3-1 -> 5-1
- J1 pad 3: 5-1 -> 3.3-1
- J10 pad 1: 3.3-2 -> 5-1
- J10 pad 3: 5-1 -> 3.3-2
- J11 pad 1: 3.3-2 -> 5-1
- J11 pad 3: 5-1 -> 3.3-2
- J12 pad 1: 3.3-2 -> 5-1
- J12 pad 3: 5-1 -> 3.3-2
- J13 pad 1: 3.3-2 -> 5-1
- J13 pad 3: 5-1 -> 3.3-2
- J14 pad 1: 3.3-2 -> 5-1
- J14 pad 3: 5-1 -> 3.3-2
- J15 pad 1: 3.3-2 -> 5-1
- J15 pad 3: 5-1 -> 3.3-2
- J16 pad 1: 3.3-2 -> 5-1
- J16 pad 3: 5-1 -> 3.3-2
- J2 pad 1: 3.3-1 -> 5-1
- J2 pad 3: 5-1 -> 3.3-1
- J3 pad 1: 3.3-1 -> 5-1
- J3 pad 3: 5-1 -> 3.3-1
- J4 pad 1: 3.3-1 -> 5-1
- J4 pad 3: 5-1 -> 3.3-1
- J5 pad 1: 3.3-1 -> 5-1
- J5 pad 3: 5-1 -> 3.3-1
- J6 pad 1: 3.3-1 -> 5-1
- J6 pad 3: 5-1 -> 3.3-1
- J7 pad 1: 3.3-1 -> 5-1
- J7 pad 3: 5-1 -> 3.3-1
- J8 pad 1: 3.3-1 -> 5-1
- J8 pad 3: 5-1 -> 3.3-1
- J9 pad 1: 3.3-2 -> 5-1
- J9 pad 3: 5-1 -> 3.3-2
- NT1 pad 2: Net-(NT1-B) -> 5-1
- U4 pad 4: Net-(NT1-A) -> Net-(U4-out+)
- U5 pad 2: 5-1 -> Net-(NT1-A)
- U5 pad 3: Net-(NT1-B) -> Net-(U4-out+)
Routing:
- net +BATT: track 0.00 -> 19.2 mm
- net Net-(J32-Pin_2): track 0.00 -> 12.7 mm
- added copper zone on F.Cu, net 14-3
- added copper zone on B.Cu, net GND
Other:
- board outline added: 95.2 x 72.4 mm

Commit message: change schematic and start layout
Parts:
- removed FID9: jumper, 218-pdb:jumper
- added C7: 0.1 uF, Capacitor_THT:C_Disc_D3.0mm_W2.0mm_P2.50mm, F.Cu at (146.0, 91.4)
- added C8: 10 uF, Capacitor_THT:C_Disc_D3.8mm_W2.6mm_P2.50mm, F.Cu at (146.0, 79.4)
- added C9: 10 uF, Capacitor_THT:C_Disc_D3.8mm_W2.6mm_P2.50mm, F.Cu at (94.6, 81.3)
- added D10: diode, >=2 Amp, Diode_THT:D_DO-15_P2.54mm_Vertical_AnodeUp, F.Cu at (153.7, 96.5)
- added FID5: jumper, 218-pdb:jumper, F.Cu at (162.6, 79.4)
- added FID6: jumper, 218-pdb:jumper, F.Cu at (162.6, 82.4)
- added R6: 1k, Resistor_THT:R_Axial_DIN0309_L9.0mm_D3.2mm_P2.54mm_Vertical, F.Cu at (159.4, 59.7)
- added TP5-1,2: TestPoint, TestPoint:TestPoint_THTPad_D2.0mm_Drill1.0mm, F.Cu at (145.4, 105.4)
- added TP5-3: TestPoint, TestPoint:TestPoint_THTPad_D2.0mm_Drill1.0mm, F.Cu at (94.6, 87.0)
- added U6: TLV76150DCY, Package_TO_SOT_SMD:SOT-223-3_TabPin2, F.Cu at (152.4, 81.3)
- D6: value diode, >=2 Amp -> LED; footprint Diode_THT:D_DO-15_P2.54mm_Vertical_AnodeUp -> 218-pdb:LED_D3.0mm
- FID10: moved to F.Cu
- NT1: value ~ -> SW_Slide_DPDT; footprint 218-pdb:PinHeader_1x03_P2.54mm_Vertical -> 218-pdb:PinHeader_2x03_P2.54mm_Vertical
- SW1: footprint 218-pdb:SLW-12689-4A-N-D -> 218-pdb:1101A4CQEA
- U1, U3: value LD1117V33 -> TLV76133DCY; footprint 218-pdb:TO255P1020X450X1968-3 -> Package_TO_SOT_SMD:SOT-223-3_TabPin2
- U5: value LD1117V50 -> TLV76150DCY; footprint 218-pdb:TO255P1020X450X1968-3 -> Package_TO_SOT_SMD:SOT-223-3_TabPin2
- moved D4 149.5 mm to (153.7, 73.7)
- moved R4 148.1 mm to (159.4, 72.4), turned to -90 degrees
- moved NT1 122.8 mm to (160.0, 82.2), turned to 90 degrees
- moved J27 114.2 mm to (172.1, 80.6), turned to 180 degrees
- moved TP1 106.0 mm to (78.1, 92.1)
- moved C6 105.8 mm to (146.0, 83.2), turned to 180 degrees
- moved C5 105.4 mm to (146.0, 87.6), turned to 180 degrees
- moved U5 95.8 mm to (152.4, 89.5), turned to 0 degrees
- moved D2 90.1 mm to (153.7, 61.0)
- moved D5 67.4 mm to (86.4, 54.0)
- moved D6 66.6 mm to (95.2, 118.7)
- moved R2 62.3 mm to (78.7, 59.7), turned to -90 degrees
- moved SW1 37.1 mm to (161.0, 89.5), turned to -90 degrees
- moved FID10 19.8 mm to (144.8, 97.8), turned to 0 degrees
- moved NT2 19.8 mm to (144.8, 95.2)
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Connections:
- C3 pad 1: 5-1 -> 5-2
- C5 pad 1: Net-(NT1-A) -> Net-(U5-VO)
- D2 pad 2: 5-2 -> 5-1
- D4 pad 2: 5-1 -> 5-2
- D5 pad 2: 14-3 -> 5-3
- D6 pad 1: 14-1 -> Net-(D6-K)
- J10 pad 1: 5-1 -> 5-2
- J11 pad 1: 5-1 -> 5-2
- J12 pad 1: 5-1 -> 5-2
- J13 pad 1: 5-1 -> 5-2
- J14 pad 1: 5-1 -> 5-2
- J15 pad 1: 5-1 -> 5-2
- J16 pad 1: 5-1 -> 5-2
- J17 pad 2: 5-2 -> 5-3
- J18 pad 2: 5-2 -> 5-3
- J19 pad 2: 5-2 -> 5-3
- J20 pad 2: 5-2 -> 5-3
- J21 pad 2: 5-2 -> 5-3
- J22 pad 2: 5-2 -> 5-3
- J23 pad 2: 5-2 -> 5-3
- J24 pad 2: 5-2 -> 5-3
- J9 pad 1: 5-1 -> 5-2
- NT1 pad 1: Net-(NT1-A) -> Net-(U6-VO)
- NT1 pad 2: 5-1 -> 5-2
- R2 pad 1: Net-(D2-K) -> Net-(D5-K)
- R5 pad 1: Net-(D5-K) -> Net-(D6-K)
- SW1 pad 1: +BATT -> 14-1
- SW1 pad 2: 14-1 -> +BATT
- U2 pad 4: 5-2 -> 5-3
- U3 pad 3: 5-1 -> 5-2
- U5 pad 2: Net-(NT1-A) -> Net-(U5-VO)
Routing:
- net +BATT: track 19.2 -> 0.00 mm
- net Net-(J32-Pin_2): track 12.7 -> 0.00 mm
Other:
- board size 95.2 x 72.4 mm -> 97.8 x 72.4 mm
