File: kicad/218-pdb.kicad_pcb (KiCad board)
At the start: 2 copper layers, 97.8 x 72.4 mm, 79 parts, among them J1 Conn_01x03, J10 Conn_01x03, J11 Conn_01x03, J12 Conn_01x03, J13 Conn_01x03, J14 Conn_01x03, J15 Conn_01x03, J16 Conn_01x03, J17 Conn_01x03, J18 Conn_01x03, J19 Conn_01x03, J2 Conn_01x03, J20 Conn_01x03, J21 Conn_01x03, J22 Conn_01x03, J23 Conn_01x03, J24 Conn_01x03, J25 Conn_01x04_Pin, J26 Conn_01x04_Pin, J27 external 5V, J28 battery, J29 battery, J3 Conn_01x03, J30 battery, J31 battery, J32 battery, J33 battery, J4 Conn_01x03, J5 Conn_01x03, J6 Conn_01x03, J7 Conn_01x03, J8 Conn_01x03, J9 Conn_01x03, SW1 5V switch, U1 TLV76133DCY, U2 DC-DC buck, U3 TLV76133DCY, U4 DC-DC buck, U5 TLV76150DCY, U6 TLV76150DCY

Commit message: edit switch
Parts:
- moved D5 66.0 mm to (86.4, 120.0)
- moved R2 50.9 mm to (92.7, 108.6), turned to 90 degrees
- moved TP1 2.62 mm to (78.7, 89.5)
- moved FID1 1.91 mm to (97.2, 86.3)
- moved FID2 1.91 mm to (137.8, 86.3)
- moved FID3 1.91 mm to (137.8, 99.0)
- moved FID4 1.91 mm to (97.2, 99.0)
- moved U2 1.91 mm to (117.5, 85.0)
- moved U4 1.91 mm to (117.5, 100.3)
- moved C9 1.91 mm to (92.7, 81.2)
- moved TP5-3 1.91 mm to (92.7, 86.9)
- moved J25 1.42 mm to (78.7, 106.0)
- moved J26 1.42 mm to (78.7, 75.6)
- moved R5 0.90 mm to (95.2, 113.0)
Changed lines of the file:
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@@
 	(footprint "Resistor_THT:R_Axial_DIN0309_L9.0mm_D3.2mm_P2.54mm_Vertical"
 		(layer "F.Cu")
-		(at 78.74 59.69 -90)
+		(at 92.71 108.585 90)
 		(descr "Resistor, Axial_DIN0309 series, Axial, Vertical, pin pitch=2.54mm, 0.5W = 1/2W, length*diameter=9*3.2mm^2, http://cdn-reichelt.de/documents/datenblatt/B400/1_4W%23YAG.pdf")
 		(tags "Resistor Axial_DIN0309 series Axial Vertical pin pitch 2.54mm 0.5W = 1/2W length 9mm diameter 3.2mm")
@@
 		)
 		(property "Manufacturer_Name" "any"
-			(at 0 0 270)
+			(at 0 0 90)
 			(unlocked yes)
 			(layer "F.Fab")
@@
 		)
 		(property "digikey_part_number" "n/a"
-			(at 0 0 270)
+			(at 0 0 90)
 			(unlocked yes)
 			(layer "F.Fab")
@@
 		)
 		(property "mount_type" "tht"
-			(at 0 0 270)
+			(at 0 0 90)
 			(unlocked yes)
 			(layer "F.Fab")
@@
 		)
 		(property "Part_Number" "spdl"
-			(at 0 0 270)
+			(at 0 0 90)
 			(unlocked yes)
 			(layer "F.Fab")
@@
 		)
 		(property "Check_prices" ""
-			(at 0 0 270)
+			(at 0 0 90)
 			(unlocked yes)
 			(layer "F.Fab")
@@
 		)
 		(property "Description_1" ""
-			(at 0 0 270)
+			(at 0 0 90)
 			(unlocked yes)
 			(layer "F.Fab")
@@
 		)
 		(property "DigiKey_Part_Number" ""
-			(at 0 0 270)
+			(at 0 0 90)
 			(unlocked yes)
 			(layer "F.Fab")
@@
 		)
 		(property "MANUFACTURER" ""
-			(at 0 0 270)
+			(at 0 0 90)
 			(unlocked yes)
 			(layer "F.Fab")
@@
 		)
 		(property "MAXIMUM_PACKAGE_HEIGHT" ""
-			(at 0 0 270)
+			(at 0 0 90)
 			(unlocked yes)
 			(layer "F.Fab")
@@
 		)
 		(property "MF" ""
-			(at 0 0 270)
+			(at 0 0 90)
 			(unlocked yes)
 			(layer "F.Fab")
@@
 		)
 		(property "MP" ""
-			(at 0 0 270)
+			(at 0 0 90)
 			(unlocked yes)
 			(layer "F.Fab")
@@
 		)
 		(property "PARTREV" ""
-			(at 0 0 270)
+			(at 0 0 90)
 			(unlocked yes)
 			(layer "F.Fab")
@@
 		)
 		(property "Package" ""
-			(at 0 0 270)
+			(at 0 0 90)
 			(unlocked yes)
 			(layer "F.Fab")
@@
 		)
 		(property "STANDARD" ""
-			(at 0 0 270)
+			(at 0 0 90)
 			(unlocked yes)
 			(layer "F.Fab")
@@
 		)
 		(property "SnapEDA_Link" ""
-			(at 0 0 270)
+			(at 0 0 90)
 			(unlocked yes)
 			(layer "F.Fab")
@@
 		)
 		(pad "1" thru_hole circle
-			(at 0 0 270)
+			(at 0 0 90)
 			(size 1.6 1.6)
 			(drill 0.8)
@@
 		)
 		(pad "2" thru_hole circle
-			(at 2.54 0 270)
+			(at 2.54 0 90)
 			(size 1.6 1.6)
 			(drill 0.8)
@@
 	(footprint "Resistor_THT:R_Axial_DIN0309_L9.0mm_D3.2mm_P2.54mm_Vertical"
 		(layer "F.Cu")
-		(at 95.885 112.395)
+		(at 95.25 113.03)
 		(descr "Resistor, Axial_DIN0309 series, Axial, Vertical, pin pitch=2.54mm, 0.5W = 1/2W, length*diameter=9*3.2mm^2, http://cdn-reichelt.de/documents/datenblatt/B400/1_4W%23YAG.pdf")
 		(tags "Resistor Axial_DIN0309 series Axial Vertical pin pitch 2.54mm 0.5W = 1/2W length 9mm diameter 3.2mm")
@@
 	(footprint "218-pdb:PinHeader_1x01_P2.54mm_H"
 		(layer "F.Cu")
-		(at 99.06 86.36 -90)
+		(at 97.154854 86.30496 -90)
 		(descr "Through hole angled pin header, 1x01, 2.54mm pitch, 6mm pin length, single row")
 		(tags "Through hole angled pin header THT 1x01 2.54mm single row")
@@
 	(footprint "Capacitor_THT:C_Disc_D3.8mm_W2.6mm_P2.50mm"
 		(layer "F.Cu")
-		(at 94.615 81.28 90)
+		(at 92.709854 81.22496 90)
 		(descr "C, Disc series, Radial, pin pitch=2.50mm, diameter*width=3.8*2.6mm^2, Capacitor, http://www.vishay.com/docs/45233/krseries.pdf")
 		(tags "C Disc series Radial pin pitch 2.50mm diameter 3.8mm width 2.6mm Capacitor")
@@
 		(tags "Switch")
 		(property "Reference" "SW1"
-			(at 0 -6.604 90)
+			(at 0 -6.604 270)
 			(layer "F.SilkS")
 			(effects
@@
 		)
 		(property "Value" "5V switch"
-			(at 0 -4.7 90)
+			(at 0 -4.7 270)
 			(layer "F.SilkS")
 			(hide yes)
@@
 		)
 		(property "Datasheet" "https://www.digikey.com/en/products/detail/cit-relay-and-switch/1101A4CQEA/20512089"
-			(at 0 0 90)
+			(at 0 0 270)
 			(layer "F.Fab")
 			(hide yes)
@@
 		)
 		(property "Description" "4.7 mm pitch"
-			(at 0 0 90)
+			(at 0 0 270)
 			(layer "F.Fab")
 			(hide yes)
@@
 			)
 		)
-		(property "Check_prices" ""
-			(at 0 0 270)
-			(unlocked yes)
-			(layer "F.Fab")
-			(hide yes)
-			(effects
-				(font
-					(size 1 1)
-					(thickness 0.15)
-				)
-			)
-		)
-		(property "Description_1" ""
-			(at 0 0 270)
-			(unlocked yes)
-			(layer "F.Fab")
-			(hide yes)
-			(effects
-				(font
-					(size 1 1)
-					(thickness 0.15)
-				)
-			)
-		)
-		(property "DigiKey_Part_Number" ""
-			(at 0 0 270)
-			(unlocked yes)
-			(layer "F.Fab")
-			(hide yes)
-			(effects
-				(font
-					(size 1 1)
-					(thickness 0.15)
-				)
-			)
-		)
-		(property "MANUFACTURER" ""
-			(at 0 0 270)
-			(unlocked yes)
-			(layer "F.Fab")
-			(hide yes)
-			(effects
-				(font
-					(size 1 1)
-					(thickness 0.15)
-				)
-			)
-		)
-		(property "MAXIMUM_PACKAGE_HEIGHT" ""
-			(at 0 0 270)
-			(unlocked yes)
-			(layer "F.Fab")
-			(hide yes)
-			(effects
-				(font
-					(size 1 1)
-					(thickness 0.15)
-				)
-			)
-		)
-		(property "MF" ""
-			(at 0 0 270)
-			(unlocked yes)
-			(layer "F.Fab")
-			(hide yes)
-			(effects
-				(font
-					(size 1 1)
-					(thickness 0.15)
-				)
-			)
-		)
-		(property "MP" ""
-			(at 0 0 270)
-			(unlocked yes)
-			(layer "F.Fab")
-			(hide yes)
-			(effects
-				(font
-					(size 1 1)
-					(thickness 0.15)
-				)
-			)
-		)
-		(property "PARTREV" ""
-			(at 0 0 270)
-			(unlocked yes)
-			(layer "F.Fab")
-			(hide yes)
-			(effects
-				(font
-					(size 1 1)
-					(thickness 0.15)
-				)
-			)
-		)
-		(property "Package" ""
-			(at 0 0 270)
-			(unlocked yes)
-			(layer "F.Fab")
-			(hide yes)
-			(effects
-				(font
-					(size 1 1)
-					(thickness 0.15)
-				)
-			)
-		)
-		(property "STANDARD" ""
-			(at 0 0 270)
-			(unlocked yes)
-			(layer "F.Fab")
-			(hide yes)
-			(effects
-				(font
-					(size 1 1)
-					(thickness 0.15)
-				)
-			)
-		)
-		(property "SnapEDA_Link" ""
-			(at 0 0 270)
-			(unlocked yes)
-			(layer "F.Fab")
-			(hide yes)
-			(effects
-				(font
-					(size 1 1)
-					(thickness 0.15)
-				)
-			)
-		)
 		(sheetname "/")
 		(sheetfile "218-pdb.kicad_sch")
@@
 		)
 		(fp_text user "${REFERENCE}"
-			(at 0 -4.7 90)
+			(at 0 -4.7 270)
 			(layer "F.Fab")
 			(effects
@@
 			)
 		)
+		(pad "" thru_hole circle
+			(at 0 -9.4 270)
+			(size 2.775 2.775)
+			(drill 1.85)
+			(layers "*.Cu" "*.Mask")
+			(remove_unused_layers no)
+		)
 		(pad "1" thru_hole rect
 			(at 0 0 270)
-			(size 2.775 2.775)
+			(size 2.9 2.9)
 			(drill 1.85)
 			(layers "*.Cu" "*.Mask")
@@
 		(pad "2" thru_hole circle
 			(at 0 -4.7 270)
-			(size 2.775 2.775)
+			(size 3 3)
 			(drill 1.85)
 			(layers "*.Cu" "*.Mask")
@@
 			(pintype "passive")
 		)
-		(pad "3" thru_hole circle
-			(at 0 -9.4 270)
-			(size 2.775 2.775)
-			(drill 1.85)
-			(layers "*.Cu" "*.Mask")
-			(remove_unused_layers no)
-		)
 		(embedded_fonts no)
 		(embedded_files
@@
 	(footprint "218-pdb:HW-411"
 		(layer "F.Cu")
-		(at 119.38 100.33)
+		(at 117.474854 100.27496)
 		(property "Reference" "U4"
 			(at 0 -0.635 0)
@@
 	(footprint "218-pdb:PinHeader_1x01_P2.54mm_H"
 		(layer "F.Cu")
-		(at 139.7 99.06 90)
+		(at 137.794854 99.00496 90)
 		(descr "Through hole angled pin header, 1x01, 2.54mm pitch, 6mm pin length, single row")
 		(tags "Through hole angled pin header THT 1x01 2.54mm single row")
@@
 	(footprint "218-pdb:LED_D3.0mm"
 		(layer "F.Cu")
-		(at 86.36 53.975)
+		(at 86.36 120.015)
 		(descr "LED, diameter 3.0mm, 2 pins, generated by kicad-footprint-generator")
 		(tags "LED")
@@
 	(footprint "218-pdb:PinHeader_1x01_P2.54mm_H"
 		(layer "F.Cu")
-		(at 99.06 99.06 90)
+		(at 97.154854 99.00496 90)
 		(descr "Through hole angled pin header, 1x01, 2.54mm pitch, 6mm pin length, single row")
 		(tags "Through hole angled pin header THT 1x01 2.54mm single row")
@@
 	(footprint "218-pdb:PinHeader_1x01_P2.54mm_H"
 		(layer "F.Cu")
-		(at 139.7 86.36 -90)
+		(at 137.794854 86.30496 -90)
 		(descr "Through hole angled pin header, 1x01, 2.54mm pitch, 6mm pin length, single row")
 		(tags "Through hole angled pin header THT 1x01 2.54mm single row")
@@
 	(footprint "Connector_PinHeader_2.54mm:PinHeader_1x04_P2.54mm_Vertical"
 		(layer "F.Cu")
-		(at 78.105 74.295 180)
+		(at 78.74 75.565 180)
 		(descr "Through hole straight pin header, 1x04, 2.54mm pitch, single row")
 		(tags "Through hole pin header THT 1x04 2.54mm single row")
@@
 	(footprint "TestPoint:TestPoint_THTPad_D2.0mm_Drill1.0mm"
 		(layer "F.Cu")
-		(at 94.615 86.995)
+		(at 92.709854 86.93996)
 		(descr "THT pad as test Point, diameter 2.0mm, hole diameter 1.0mm")
 		(tags "test point THT pad")
@@
 	(footprint "Connector_PinHeader_2.54mm:PinHeader_1x04_P2.54mm_Vertical"
 		(layer "F.Cu")
-		(at 78.105 107.315 180)
+		(at 78.74 106.045 180)
 		(descr "Through hole straight pin header, 1x04, 2.54mm pitch, single row")
 		(tags "Through hole pin header THT 1x04 2.54mm single row")
@@
 	(footprint "218-pdb:HW-411"
 		(layer "F.Cu")
-		(at 119.38 85.09 180)
+		(at 117.474854 85.03496 180)
 		(property "Reference" "U2"
 			(at 0 -0.635 0)
@@
 	(footprint "TestPoint:TestPoint_Bridge_Pitch5.08mm_Drill0.7mm"
 		(layer "F.Cu")
-		(at 78.105 92.075 90)
+		(at 78.74 89.535 90)
 		(descr "wire loop as test point, pitch 5.08mm, hole diameter 0.7mm, wire diameter 1.0mm")
 		(tags "test point wire loop")

Commit message: add traces
Parts:
- added G***: LOGO, LOGO, B.Cu at (117.6, 92.6)
- moved TP5-1,2 52.8 mm to (92.7, 101.6)
- moved D10 9.52 mm to (144.1, 96.5), turned to 0 degrees
- moved NT2 7.85 mm to (142.9, 102.9), turned to 90 degrees
- moved FID10 5.12 mm to (145.4, 102.9), turned to 90 degrees
- moved C2 3.20 mm to (166.4, 54.2), turned to 180 degrees
- moved TP5-3 2.48 mm to (92.7, 84.5)
- moved R2 2.41 mm to (92.7, 106.2), turned to -90 degrees
- moved C4 2.17 mm to (167.9, 66.7), turned to 0 degrees
- moved J27 0.66 mm to (172.1, 81.3)
- moved C9 0.06 mm to (92.7, 81.3)
- renumbered C8 to C5, C7 to C6, C6 to C7, C5 to C8, U6 to U5, U5 to U6
Connections:
- C5 pad 1: Net-(U6-VO) -> Net-(U5-VO)
- C8 pad 1: Net-(U5-VO) -> Net-(U6-VO)
- R2 pad 1: Net-(D5-K) -> GND
- R2 pad 2: GND -> Net-(D5-K)
- U5 pad 2: Net-(U6-VO) -> Net-(U5-VO)
- U6 pad 2: Net-(U5-VO) -> Net-(U6-VO)
Routing:
- net 14-1: track 0.00 -> 102.1 mm
- net 5-1: track 0.00 -> 92.8 mm
- net 5-2: track 0.00 -> 86.5 mm
- net 3.3-2: track 0.00 -> 83.1 mm
- net 3.3-1: track 0.00 -> 82.7 mm
- net Net-(U4-out+): track 0.00 -> 81.6 mm
- net 5-3: track 0.00 -> 81.3 mm
- net +BATT: track 0.00 -> 39.6 mm
- net 14-3: track 0.00 -> 26.5 mm, vias 0 -> 1
- net 14-2: track 0.00 -> 25.4 mm
- net Net-(U6-VO): track 0.00 -> 19.6 mm
- net Net-(U5-VO): track 0.00 -> 15.7 mm
- net Net-(D5-K): track 0.00 -> 13.9 mm
- net Net-(J32-Pin_2): track 0.00 -> 12.7 mm
- net Net-(J27-Pin_2): track 0.00 -> 10.1 mm
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- added copper zone on F.Cu, net +BATT
- added copper zone on F.Cu, net 3.3-1
- added copper zone on F.Cu, net 3.3-2
- added copper zone on F.Cu, net GND
- added copper zone on F.Cu, net Net-(U5-VO)
- added copper zone on F.Cu, net Net-(U6-VO)
Other:
- outline, holes or cut-outs redrawn
- board text added: "PDB"
- board text added: "SPDL"
- board text added: "V2.1, 2026, JLP"
- board text added: "github.com/SPDLDaemon/SPDL-PDB"
