File: kicad/218-pdb.kicad_pcb (KiCad board)
At the start: 2 copper layers, 97.8 x 72.4 mm, 80 parts, among them J1 Conn_01x03, J10 Conn_01x03, J11 Conn_01x03, J12 Conn_01x03, J13 Conn_01x03, J14 Conn_01x03, J15 Conn_01x03, J16 Conn_01x03, J17 Conn_01x03, J18 Conn_01x03, J19 Conn_01x03, J2 Conn_01x03, J20 Conn_01x03, J21 Conn_01x03, J22 Conn_01x03, J23 Conn_01x03, J24 Conn_01x03, J25 Conn_01x04_Pin, J26 Conn_01x04_Pin, J27 external 5V, J28 battery, J29 battery, J3 Conn_01x03, J30 battery, J31 battery, J32 battery, J33 battery, J4 Conn_01x03, J5 Conn_01x03, J6 Conn_01x03, J7 Conn_01x03, J8 Conn_01x03, J9 Conn_01x03, SW1 5V switch, U1 TLV76133DCY, U2 DC-DC buck, U3 TLV76133DCY, U4 DC-DC buck, U5 TLV76150DCY, U6 TLV76150DCY

Commit message: update bom
Parts:
- J28, J29, J30, J31: value battery -> 14v
- moved R2 2.29 mm to (92.6, 108.5)
- moved R5 2.01 mm to (97.2, 112.4), turned to 90 degrees
- moved main1 1.91 mm to (151.1, 114.9)
- moved SW1 0.66 mm to (161.0, 88.9)
- moved J27 0.27 mm to (172.1, 81.0)
Routing:
- net +BATT: track 39.6 -> 28.3 mm
- net Net-(D5-K): track 13.9 -> 11.6 mm
- net Net-(D6-K): track 5.72 -> 7.16 mm
Other:
- board text added: "+5V-"
- board text added: "- +"
- board text added: "1 2 3 4 5 6 7 8"
- board text added: "14V"
- board text added: "5-1"
- board text added: "5-2"
- board text added: "5V switch"
- board text added: "NT2"
- board text added: "V2.1, 2026, Joshua"
- board text added: "bat"
- board text added: "batteries"
- board text added: "ext"
- board text added: "switch and fuse"
- board text removed: "V2.1, 2026, JLP"

Commit message: adjust layout
Other:
- board text added: "main switch"
- board text added: "servo pwr"
Changed lines of the file:
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@@
+		)
+	)
+	(gr_text "5V switch"
+		(at 150.876 106.426 90)
+		(layer "F.SilkS")
+		(effects
+			(font
+				(size 1 1)
+				(thickness 0.125)
+			)
+			(justify left bottom)
 		)
 	)
@@
 	(gr_text "5V switch"
 		(at 158.965222 92.587559 90)
+		(layer "F.SilkS")
+		(effects
+			(font
+				(size 1 1)
+				(thickness 0.125)
+			)
+			(justify left bottom)
+		)
+	)
+	(gr_text "servo pwr"
+		(at 141.695133 101.390694 0)
+		(layer "F.SilkS")
+		(effects
+			(font
+				(size 1 1)
+				(thickness 0.125)
+			)
+			(justify left bottom)
+		)
+	)
+	(gr_text "main switch"
+		(at 141.3746 107.416716 90)
 		(layer "F.SilkS")
 		(effects
@@
 		(polygon
 			(pts
-				(xy 100.457 107.95) (xy 100.457 123.19) (xy 173.99 123.19) (xy 173.99 93.345) (xy 156.21 93.345)
-				(xy 156.21 97.79) (xy 146.05 107.95)
+				(xy 100.457 107.95) (xy 100.457 123.19) (xy 173.99 123.19) (xy 173.99 93.345) (xy 165.227 93.345)
+				(xy 165.227 93.840573) (xy 152.019 93.853) (xy 152.019 101.981) (xy 146.05 107.95)
 			)
 		)
@@
 			(pts
 				(xy 173.99 50.8) (xy 76.2 50.8) (xy 76.2 123.19) (xy 100.203 123.19) (xy 100.203 107.696) (xy 145.669 107.696)
-				(xy 156.464 96.901) (xy 156.464 93.599) (xy 173.99 93.599)
-			)
-		)
+				(xy 151.638 101.727) (xy 151.638 93.599) (xy 173.99 93.599)
+			)
+		)

Commit message: work on diagram and silkscreen
Parts:
- moved D6 1.25 mm to (95.2, 120.0)
Routing:
- net Net-(D6-K): track 7.16 -> 8.42 mm
- net 14-3: track 26.5 -> 27.0 mm
Other:
- board text added: "3 G 5"
- board text added: "3.3-1"
- board text added: "3.3-2"
Changed lines of the file:
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@@
 	(footprint "218-pdb:LED_D3.0mm"
 		(layer "F.Cu")
-		(at 95.25 118.745)
+		(at 95.229223 119.997066)
 		(descr "LED, diameter 3.0mm, 2 pins, generated by kicad-footprint-generator")
 		(tags "LED")
@@
 	(footprint "218-pdb:LED_D3.0mm"
 		(layer "F.Cu")
-		(at 86.36 120.015)
+		(at 86.346373 119.997066)
 		(descr "LED, diameter 3.0mm, 2 pins, generated by kicad-footprint-generator")
 		(tags "LED")
@@
 		(layer "Edge.Cuts")
 	)
+	(gr_text "5-1"
+		(at 153.156141 64.00398 0)
+		(layer "F.SilkS")
+		(effects
+			(font
+				(size 1 1)
+				(thickness 0.125)
+			)
+			(justify left bottom)
+		)
+	)
+	(gr_text "3\n\nG\n\n5"
+		(at 90.296755 62.1568 0)
+		(layer "F.SilkS")
+		(effects
+			(font
+				(size 1.1 1.2)
+				(thickness 0.2)
+				(bold yes)
+			)
+			(justify left bottom)
+		)
+	)
 	(gr_text "ext"
 		(at 164.737961 77.662475 0)
@@
 		)
 	)
+	(gr_text "3.3-1"
+		(at 151.992766 52.697432 0)
+		(layer "F.SilkS")
+		(effects
+			(font
+				(size 1 1)
+				(thickness 0.125)
+			)
+			(justify left bottom)
+		)
+	)
 	(gr_text "5-2"
 		(at 160.865981 84.947011 0)
@@
 		)
 	)
+	(gr_text "3.3-2"
+		(at 151.992766 65.385487 0)
+		(layer "F.SilkS")
+		(effects
+			(font
+				(size 1 1)
+				(thickness 0.125)
+			)
+			(justify left bottom)
+		)
+	)
+	(gr_text "3\n\nG\n\n5"
+		(at 90.406066 75.168507 0)
+		(layer "F.SilkS")
+		(effects
+			(font
+				(size 1.1 1.2)
+				(thickness 0.2)
+				(bold yes)
+			)
+			(justify left bottom)
+		)
+	)
 	(gr_text "5V switch"
 		(at 158.965222 92.587559 90)
@@
 		)
 	)
+	(gr_text "5-2"
+		(at 153.284361 76.818531 0)
+		(layer "F.SilkS")
+		(effects
+			(font
+				(size 1 1)
+				(thickness 0.125)
+			)
+			(justify left bottom)
+		)
+	)
 	(gr_text "- +"
 		(at 170.551801 94.989027 270)
@@
 	)
 	(segment
-		(start 97.79 118.745)
+		(start 99.021289 118.745)
 		(end 104.08973 118.745)
 		(width 0.25)
@@
 	)
 	(segment
+		(start 97.769223 119.997066)
+		(end 99.021289 118.745)
+		(width 0.25)
+		(layer "F.Cu")
+		(net 13)
+	)
+	(segment
 		(start 146.685 96.52)
 		(end 146.05 97.155)
@@
 	)
 	(segment
-		(start 86.36 120.015)
+		(start 86.377934 119.997066)
 		(end 91.694 114.681)
 		(width 0.25)
@@
 	)
 	(segment
+		(start 91.694 111.887)
+		(end 92.583 110.998)
+		(width 0.25)
+		(layer "F.Cu")
+		(net 24)
+	)
+	(segment
 		(start 91.694 114.681)
 		(end 91.694 111.887)
@@
 	)
 	(segment
-		(start 91.694 111.887)
-		(end 92.583 110.998)
+		(start 86.346373 119.997066)
+		(end 86.377934 119.997066)
 		(width 0.25)
 		(layer "F.Cu")
@@
 	)
 	(segment
-		(start 87.63 121.285)
-		(end 85.178 121.285)
+		(start 88.9 120.015)
+		(end 87.503 121.412)
 		(width 0.25)
 		(layer "F.Cu")
@@
 	)
 	(segment
-		(start 97.154854 80.58996)
-		(end 97.099814 80.645)
-		(width 1.25)
+		(start 84.836 121.0505)
+		(end 84.836 114.554)
+		(width 0.25)
 		(layer "F.Cu")
 		(net 27)
 	)
 	(segment
-		(start 85.725 60.325)
-		(end 85.725 113.665)
-		(width 1)
+		(start 85.1975 121.412)
+		(end 84.836 121.0505)
+		(width 0.25)
 		(layer "F.Cu")
 		(net 27)
 	)
 	(segment
-		(start 92.71 84.455)
-		(end 92.71 81.28)
-		(width 0.25)
+		(start 97.154854 80.58996)
+		(end 97.099814 80.645)
+		(width 1.25)
 		(layer "F.Cu")
 		(net 27)
 	)
 	(segment
-		(start 85.178 121.285)
-		(end 84.605 120.712)
-		(width 0.25)
+		(start 85.725 60.325)
+		(end 85.725 113.665)
+		(width 1)
 		(layer "F.Cu")
 		(net 27)
 	)
 	(segment
-		(start 84.605 114.785)
-		(end 85.725 113.665)
+		(start 87.503 121.412)
+		(end 85.1975 121.412)
 		(width 0.25)
 		(layer "F.Cu")
@@
 	)
 	(segment
-		(start 88.9 120.015)
-		(end 87.63 121.285)
+		(start 92.71 84.455)
+		(end 92.71 81.28)
 		(width 0.25)
 		(layer "F.Cu")
@@
 	)
 	(segment
-		(start 84.605 120.712)
-		(end 84.605 114.785)
+		(start 84.836 114.554)
+		(end 85.725 113.665)
 		(width 0.25)
 		(layer "F.Cu")
@@
 	(segment
 		(start 95.25 114.281)
-		(end 95.25 118.745)
+		(end 95.25 119.976289)
+		(width 0.25)
+		(layer "F.Cu")
+		(net 29)
+	)
+	(segment
+		(start 95.25 119.976289)
+		(end 95.229223 119.997066)
 		(width 0.25)
 		(layer "F.Cu")

Commit message: adjust layout
Parts:
- turned FID10 to -90 degrees
Routing:
- net +BATT: track 28.3 -> 29.2 mm
Other:
- board text added: "17 18 19 20 21 22 23 24"
- board text added: "9 10 11 12 13 14 15 16"
- board text added: "S 5V G"
Changed lines of the file:
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@@
 		(tags "Resistor Axial_DIN0309 series Axial Vertical pin pitch 2.54mm 0.5W = 1/2W length 9mm diameter 3.2mm")
 		(property "Reference" "R1"
-			(at -2.54 0 0)
+			(at -2.032 -1.778 0)
 			(layer "F.SilkS")
 			(effects
@@
 		(tags "C Disc series Radial pin pitch 2.50mm diameter 3mm width 2mm Capacitor")
 		(property "Reference" "C1"
-			(at -1.29 -1.27 180)
+			(at -1.665423 0.120084 180)
 			(layer "F.SilkS")
 			(effects
@@
 	(footprint "218-pdb:jumper"
 		(layer "F.Cu")
-		(at 145.415 102.87 90)
+		(at 145.415 102.87 -90)
 		(property "Reference" "FID10"
-			(at 0 -0.5 90)
+			(at 0 -0.5 270)
 			(unlocked yes)
 			(layer "F.SilkS")
@@
 		)
 		(property "Value" "jumper"
-			(at 0 1 90)
+			(at 0 1 270)
 			(unlocked yes)
 			(layer "F.Fab")
@@
 		)
 		(property "Datasheet" "~"
-			(at 0 0 90)
+			(at 0 0 270)
 			(unlocked yes)
 			(layer "F.Fab")
@@
 		)
 		(property "Description" "Fiducial Marker"
-			(at 0 0 90)
+			(at 0 0 270)
 			(unlocked yes)
 			(layer "F.Fab")
@@
 		)
 		(property "Part_Number" "pin jumper 0.1\" pitch Sullins QPC02SXGN-RC"
-			(at 0 0 270)
+			(at 0 0 90)
 			(unlocked yes)
 			(layer "F.Fab")
@@
 		)
 		(property "Check_prices" ""
-			(at 0 0 270)
+			(at 0 0 90)
 			(unlocked yes)
 			(layer "F.Fab")
@@
 		)
 		(property "Description_1" ""
-			(at 0 0 270)
+			(at 0 0 90)
 			(unlocked yes)
 			(layer "F.Fab")
@@
 		)
 		(property "DigiKey_Part_Number" ""
-			(at 0 0 270)
+			(at 0 0 90)
 			(unlocked yes)
 			(layer "F.Fab")
@@
 		)
 		(property "MANUFACTURER" ""
-			(at 0 0 270)
+			(at 0 0 90)
 			(unlocked yes)
 			(layer "F.Fab")
@@
 		)
 		(property "MAXIMUM_PACKAGE_HEIGHT" ""
-			(at 0 0 270)
+			(at 0 0 90)
 			(unlocked yes)
 			(layer "F.Fab")
@@
 		)
 		(property "MF" ""
-			(at 0 0 270)
+			(at 0 0 90)
 			(unlocked yes)
 			(layer "F.Fab")
@@
 		)
 		(property "MP" ""
-			(at 0 0 270)
+			(at 0 0 90)
 			(unlocked yes)
 			(layer "F.Fab")
@@
 		)
 		(property "PARTREV" ""
-			(at 0 0 270)
+			(at 0 0 90)
 			(unlocked yes)
 			(layer "F.Fab")
@@
 		)
 		(property "Package" ""
-			(at 0 0 270)
+			(at 0 0 90)
 			(unlocked yes)
 			(layer "F.Fab")
@@
 		)
 		(property "STANDARD" ""
-			(at 0 0 270)
+			(at 0 0 90)
 			(unlocked yes)
 			(layer "F.Fab")
@@
 		)
 		(property "SnapEDA_Link" ""
-			(at 0 0 270)
+			(at 0 0 90)
 			(unlocked yes)
 			(layer "F.Fab")
@@
 		)
 		(fp_text user "${REFERENCE}"
-			(at 0 2.5 90)
+			(at 0 2.5 270)
 			(unlocked yes)
 			(layer "F.Fab")
@@
 		(tags "Resistor Axial_DIN0309 series Axial Vertical pin pitch 2.54mm 0.5W = 1/2W length 9mm diameter 3.2mm")
 		(property "Reference" "R6"
-			(at -1.778 2.159 180)
+			(at -1.921237 -1.900961 180)
 			(layer "F.SilkS")
 			(effects
@@
 		(tags "C Disc series Radial pin pitch 2.50mm diameter 3mm width 2mm Capacitor")
 		(property "Reference" "C3"
-			(at 4.298 0 180)
+			(at -1.29 1.397 180)
 			(layer "F.SilkS")
 			(effects
@@
 		(tags "Resistor Axial_DIN0309 series Axial Vertical pin pitch 2.54mm 0.5W = 1/2W length 9mm diameter 3.2mm")
 		(property "Reference" "R4"
-			(at -1.778 2.159 180)
+			(at -2.032 -1.778 180)
 			(layer "F.SilkS")
 			(effects
@@
 		(tags "Switch")
 		(property "Reference" "SW1"
-			(at 0 -6.604 270)
+			(at -0.106165 -7.118209 270)
 			(layer "F.SilkS")
 			(effects
@@
 		)
 		(fp_text user "IN-\n"
-			(at -20.955 -5.08 0)
+			(at -18.160854 -0.07196 0)
 			(unlocked yes)
 			(layer "F.SilkS")
@@
 		)
 		(fp_text user "OUT-\n"
-			(at 12.7 -5.08 0)
+			(at 10.287146 -0.32596 0)
 			(unlocked yes)
 			(layer "F.SilkS")
@@
 		)
 		(fp_text user "OUT+"
-			(at 10.795 5.715 0)
+			(at 10.254946 5.727551 0)
 			(unlocked yes)
 			(layer "F.SilkS")
@@
 		(tags "Resistor Axial_DIN0309 series Axial Vertical pin pitch 2.54mm 0.5W = 1/2W length 9mm diameter 3.2mm")
 		(property "Reference" "R3"
-			(at -2.54 0 0)
+			(at -2.286 -1.27 0)
 			(layer "F.SilkS")
 			(effects
@@
 		)
 		(fp_text user "IN-\n"
-			(at -20.955 -5.08 180)
+			(at -18.542146 -0.43604 180)
 			(unlocked yes)
 			(layer "F.SilkS")
@@
 		)
 		(fp_text user "OUT-\n"
-			(at 12.7 -5.08 180)
+			(at 10.286854 -0.30904 180)
 			(unlocked yes)
 			(layer "F.SilkS")
@@
 		)
 		(fp_text user "OUT+"
-			(at 10.795 5.715 180)
+			(at 10.448322 5.688732 180)
 			(unlocked yes)
 			(layer "F.SilkS")
@@
 	)
 	(gr_line
+		(start 79.375 92.075)
+		(end 78.105 92.075)
+		(stroke
+			(width 0.1)
+			(type default)
+		)
+		(layer "F.SilkS")
+	)
+	(gr_line
+		(start 79.121 92.448988)
+		(end 78.359 92.448988)
+		(stroke
+			(width 0.1)
+			(type default)
+		)
+		(layer "F.SilkS")
+	)
+	(gr_line
 		(start 78.74 75.565)
 		(end 83.185 83.205)
@@
 	)
 	(gr_line
+		(start 78.867 92.836978)
+		(end 78.613 92.836978)
+		(stroke
+			(width 0.1)
+			(type default)
+		)
+		(layer "F.SilkS")
+	)
+	(gr_line
+		(start 93.91 84.455)
+		(end 95.25 84.455)
+		(stroke
+			(width 0.1)
+			(type default)
+		)
+		(layer "F.SilkS")
+	)
+	(gr_line
 		(start 83.185 106.045)
 		(end 78.74 103.505)
@@
 		(layer "F.SilkS")
 	)
+	(gr_line
+		(start 93.91 101.6)
+		(end 95.25 101.6)
+		(stroke
+			(width 0.1)
+			(type default)
+		)
+		(layer "F.SilkS")
+	)
+	(gr_line
+		(start 78.74 90.435)
+		(end 78.74 92.075)
+		(stroke
+			(width 0.1)
+			(type default)
+		)
+		(layer "F.SilkS")
+	)
 	(gr_arc
 		(start 173.99 120.015)
@@
 		)
 	)
+	(gr_text "17       18       19       20       21       22       23       24"
+		(at 93.574431 65.020634 0)
+		(layer "F.SilkS")
+		(effects
+			(font
+				(size 1 1.055)
+				(thickness 0.125)
+			)
+			(justify left bottom)
+		)
+	)
 	(gr_text "-  +"
 		(at 124.311966 122.537985 0)
@@
 		)
 	)
+	(gr_text "S  5V  G\n"
+		(at 82.042 56.896 0)
+		(layer "F.SilkS")
+		(effects
+			(font
+				(size 1.1 1.1)
+				(thickness 0.22)
+				(bold yes)
+			)
+			(justify left bottom)
+		)
+	)
 	(gr_text "14V"
 		(at 104.139625 122.035112 0)
@@
 	)
 	(gr_text "5V switch"
-		(at 150.876 106.426 90)
+		(at 150.749 106.426 90)
 		(layer "F.SilkS")
 		(effects
@@
 		)
 	)
+	(gr_text "9       10       11       12       13       14       15       16"
+		(at 94.102137 52.317207 0)
+		(layer "F.SilkS")
+		(effects
+			(font
+				(size 1 1.055)
+				(thickness 0.125)
+			)
+			(justify left bottom)
+		)
+	)
 	(gr_text "servo pwr"
 		(at 141.695133 101.390694 0)
@@
 	)
 	(segment
-		(start 170.434 94.234)
-		(end 170.434 108.294537)
-		(width 0.5)
+		(start 165.729791 89.529791)
+		(end 170.434 94.234)
+		(width 2)
 		(layer "F.Cu")
 		(net 9)
 	)
 	(segment
-		(start 170.434 108.294537)
+		(start 170.434 108.712)
+		(end 165.487725 113.658275)
+		(width 2)
+		(layer "F.Cu")
+		(net 9)
+	)
+	(segment
+		(start 165.487725 113.658275)
 		(end 165.070262 113.658275)
-		(width 0.5)
+		(width 2)
 		(layer "F.Cu")
 		(net 9)
 	)
 	(segment
-		(start 165.735 89.535)
-		(end 170.434 94.234)
-		(width 0.5)
+		(start 165.729791 88.879165)
+		(end 165.729791 89.529791)
+		(width 2)
+		(layer "F.Cu")
+		(net 9)
+	)
+	(segment
+		(start 170.434 94.234)
+		(end 170.434 108.712)
+		(width 2)
 		(layer "F.Cu")
 		(net 9)

Commit message: adjust layout
Parts:
- removed TP5-1,2, TP5-3: TestPoint, TestPoint:TestPoint_THTPad_D2.0mm_Drill1.0mm
- added TP-U1: TestPoint, TestPoint:TestPoint_THTPad_D2.0mm_Drill1.0mm, F.Cu at (92.7, 103.7)
- added TP-U2: TestPoint, TestPoint:TestPoint_THTPad_D2.0mm_Drill1.0mm, F.Cu at (92.7, 84.5)
- moved R2 2.67 mm to (92.7, 111.1)
- moved R5 1.25 mm to (97.1, 111.1), turned to -90 degrees
- renumbered U4 to U1, U1 to U3, U3 to U4
Connections:
- R5 pad 1: Net-(D6-K) -> GND
- R5 pad 2: GND -> Net-(D6-K)
Routing:
- net Net-(J32-Pin_2): track 12.7 -> 6.35 mm
- net +BATT: track 29.2 -> 32.3 mm
- net Net-(D5-K): track 11.6 -> 8.97 mm
- net Net-(U1-out+): track 81.6 -> 79.8 mm
- net Net-(D6-K): track 8.42 -> 7.15 mm
- added copper zone on F.Cu, net Net-(J32-Pin_2)
Other:
- board text added: "14v"
- board text added: "5-3"
